File: hardware/kicad/ReRAM-SMU-V1/sheets/07_COMPLIANCE_TRIP.kicad_sch (KiCad schematic)
At the start: 3 parts, among them U1 TLV3501 emergency supervisor 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

Commit message: hardware: pre-ERC manufacturer corrections (LT1970 physical pins, ADS1262 TSSOP-28, MCU G431RBT6, 74LVC1G74 latch, LT5400 Kelvin, AD5764 rails, ADS1262 bipolar)
Parts:
- removed R1: 10k pull-up ISRC to 3.3V PRIMARY, Resistor_SMD:R_0805_2012Metric, symbol Device:R
- removed R2: 10k pull-up ISNK to 3.3V PRIMARY, Resistor_SMD:R_0805_2012Metric, symbol Device:R
- removed U1: TLV3501 emergency supervisor ONLY 6.5mV, Package_TO_SOT_SMD:SOT-23-6, symbol Device:OpAmp
Other:
- note removed: "07_COMPLIANCE_TRIP LT1970 continuous CC via shared shunt TLV3501 loose 120-150% only ISRC/ISNK pull-ups 10k to 3.3V"
- company: ReRAM-SMU V1 -> (none)
- title: 07_COMPLIANCE_TRIP -> (none)
