File: hardware/kicad/ReRAM-SMU-V1/sheets/09_DUT_CONNECTOR_GUARD.kicad_sch (KiCad schematic)
At the start: 1 part, among them J1 DUT 4-wire Kelvin connector P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

Commit message: hardware: pre-ERC manufacturer corrections (LT1970 physical pins, ADS1262 TSSOP-28, MCU G431RBT6, 74LVC1G74 latch, LT5400 Kelvin, AD5764 rails, ADS1262 bipolar)
Parts:
- removed J1: DUT 4-wire Kelvin connector PRIMARY, Connector:Banana_Jack_4Pin, symbol Device:R
Other:
- note removed: "09_DUT_CONNECTOR_GUARD FORCE_HI/LO SENSE_HI/LO shield guard keepout ESD low-leak"
- company: ReRAM-SMU V1 -> (none)
- title: 09_DUT_CONNECTOR_GUARD -> (none)
