File: hardware/kicad/ReRAM-SMU-V1/sheets/08_MCU_USB_CONTROL.kicad_sch (KiCad schematic)
At the start: 1 part, among them U1 STM32G474 PRIMARY LQFP-64

Commit message: hardware: pre-ERC manufacturer corrections (LT1970 physical pins, ADS1262 TSSOP-28, MCU G431RBT6, 74LVC1G74 latch, LT5400 Kelvin, AD5764 rails, ADS1262 bipolar)
Parts:
- removed U1: STM32G474 PRIMARY LQFP-64, Package_QFP:LQFP-64_10x10mm_P0.5mm, symbol Device:OpAmp
Other:
- note removed: "08_MCU_USB_CONTROL STM32G4 USB-C relay drivers watchdog supervisor Safe POR ENABLE"
- company: ReRAM-SMU V1 -> (none)
- title: 08_MCU_USB_CONTROL -> (none)
