File: hardware/kicad/ReRAM-SMU-V1/sheets/05_CURRENT_RANGES.kicad_sch (KiCad schematic)
At the start: 18 parts, among them K1A TQ2-5V NO 10mA 2.5R, K1B REED SENSE K1 <1pA, K2A TQ2-5V NO 1mA 25R, K2B REED SENSE K2, K3A TQ2-5V NO 100uA 499R, K3B REED SENSE K3, K4A TQ2-5V NO 10uA 4.99k, K4B REED SENSE K4, K5A Coto9007-5V NO <1pA 1uA 100k, K5B REED SENSE K5 <1pA 100k, K6A Coto9007-5V *NC* <1pA SAFE DE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, K6B REED SENSE *NC* SAFE 1M

Commit message: style(kicad): re-serialize 01-06 + root to KiCad 9.0 schema 20250114 (formatting only)
- (version 20241014)->(version 20250114) + generator_version 10.0->9.0 on all 10 sch files including root + 01-04 verified via git diff
- lib_symbols block pretty-print expansion: property/symbol multi-line with explicit hide/exclude/effects font, no wire/symbol/net deletion
- 8 files: ReRAM-SMU-V1.kicad_pro (453+9-), ReRAM-SMU-V1.kicad_sch (806+53-), 01_POWER (5724+411-), 02_DAC (5816+436-), 03_OUTPUT (4308+276-), 04_KELVIN (3720+270-), 05_CURRENT_RANGES (375+217-), 06_ADC (492+452-); total 21694+2124-
- 07/08/09 excluded (already restored 184/236/156 lines, verified not truncated; no re-serialization needed)
- Functional audit: no net/junction/wire loss, netlist continuity preserved, ERC 124 headless (ca7eac3) unchanged by re-serialization
- Verified: wc -l 01 5739,02 5831,03 4322,04 3735,05 388,06 507,07 184,08 236,09 156
Parts:
- removed K1A: TQ2-5V NO 10mA 2.5R, Relay_THT:TQ2-5V, symbol Custom:REED_RELAY_SPST
- removed K1B: REED SENSE K1 <1pA, symbol Custom:REED_RELAY_SPST
- removed K2A: TQ2-5V NO 1mA 25R, symbol Custom:REED_RELAY_SPST
- removed K2B: REED SENSE K2, symbol Custom:REED_RELAY_SPST
- removed K3A: TQ2-5V NO 100uA 499R, symbol Custom:REED_RELAY_SPST
- removed K3B: REED SENSE K3, symbol Custom:REED_RELAY_SPST
- removed K4A: TQ2-5V NO 10uA 4.99k, symbol Custom:REED_RELAY_SPST
- removed K4B: REED SENSE K4, symbol Custom:REED_RELAY_SPST
- removed K5A: Coto9007-5V NO <1pA 1uA 100k, Relay_THT:Coto_9007, symbol Custom:REED_RELAY_SPST
- removed K5B: REED SENSE K5 <1pA 100k, symbol Custom:REED_RELAY_SPST
- removed K6A: Coto9007-5V *NC* <1pA SAFE DEFAULT 1M 100nA, Relay_THT:Coto_9007_NC, symbol Custom:REED_RELAY_SPST_NC
- removed K6B: REED SENSE *NC* SAFE 1M, symbol Custom:REED_RELAY_SPST_NC
- removed R1: 2.49R 0.1% 25ppm 0.25W Kelvin 4-pad [2.5R nom], Resistor_SMD:R_1206_3216Metric_Kelvin, symbol Device:R
- removed R2: 24.9R 0.1% 25ppm [25R nom] 1mA 25mV, Resistor_SMD:R_0805_2012Metric, symbol Device:R
- removed R3: 499R 0.1% 25ppm [500R] 100uA 50mV, Resistor_SMD:R_0805_2012Metric, symbol Device:R
- removed R4: 4.99k 0.1% 25ppm [5k] 10uA 50mV, Resistor_SMD:R_0805_2012Metric, symbol Device:R
- removed R5: 100k 0.01% 10ppm [100k] 1uA 100mV *TIGHT*, Resistor_SMD:R_0805_2012Metric_Guard, symbol Device:R
- removed R6: 1.00M 0.01% 10ppm [1M] 100nA 100mV *TIGHT GUARD*, Resistor_SMD:R_0805_2012Metric_Guard_Keepout, symbol Device:R
Other:
- note removed: "05_CURRENT_RANGES — Gate D detailed: 6 shared low-side shunts, Kelvin taps at R pad (NOT relay pole), BBM, safe default K6 NC=1M"
- note removed: "A: 10mA 2.49R 25mV B: 1mA 24.9R 25mV C: 100uA 499R 50mV D: 10uA 4.99k 50mV E: 1uA 100k 100mV *0.01%* F: 100nA 1M 100mV *0.01% 10ppm NC SAFE* — Force relays TQ2 / Sense Coto9007 <1pA"
- note removed: "BBM: one-hot shift register + 5ms break + 10ms settle + firmware hold. NC K6/K6B de-energized default → 1M between FORCE_LO–GND"
- note removed: "KELVIN: ISENSE_P_K / ISENSE_N_K (=GND star) → 06 + LT1970 SENSE_N/P — contact R OUTSIDE sense"
- note removed: "LAYOUT: R bottoms → GND_KELVIN_STAR (4 vias, single point). Sense 0.3mm diff, no vias, guard keepout on R5/R6 (exposed copper, 0.5mm gap, stitched plane DNP). Force 0.5mm."
- note removed: "REF: GROUNDING GND-05/07 relay return to supply entry, not analog plane. Contact audit §3.2 inside/outside. Leak <1pA reed for E/F."
